File: Teensy.kicad_sch (KiCad schematic)
At the start: 12 parts

Commit message: added TVS diodes to external pins for protection. Ran fabrication output. Ran iBOM generation. All part links can be seen in the iBOM. Download and open to see this
Parts:
- B100: DIGIKEY LINK (none) -> https://www.digikey.com/en/products/detail/keystone-electro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
- D100, D101, D102: DIGIKEY LINK (none) -> https://www.digikey.com/en/products/detail/w%C3%BCrth-elekt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
- Q100: DIGIKEY LINK (none) -> https://www.digikey.com/en/products/detail/sparkfun-electro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
- R100, R101, R102, R128, R129: DIGIKEY LINK (none) -> https://www.digikey.com/en/products/detail/yageo/RC0603FR-0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
- R140, R141: DIGIKEY LINK (none) -> https://www.digikey.com/en/products/detail/yageo/RC0603JR-0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
Changed lines of the file:
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@@
 	(generator_version "8.0")
 	(paper "A4")
+	(title_block
+		(date "2025-02-11")
+	)
 	(junction
 		(at 43.18 175.26)
@@
 			)
 		)
+		(property "DIGIKEY LINK" "https://www.digikey.com/en/products/detail/yageo/RC0603JR-070RL/726675"
+			(at 99.06 114.3 0)
+			(effects
+				(font
+					(size 1.27 1.27)
+				)
+				(hide yes)
+			)
+		)
 		(pin "2"
 		)
@@
 		)
 		(property "Description" "Resistor"
+			(at 240.03 57.15 0)
+			(effects
+				(font
+					(size 1.27 1.27)
+				)
+				(hide yes)
+			)
+		)
+		(property "DIGIKEY LINK" "https://www.digikey.com/en/products/detail/yageo/RC0603FR-0710KL/726880"
 			(at 240.03 57.15 0)
 			(effects
@@
 			)
 		)
+		(property "DIGIKEY LINK" "https://www.digikey.com/en/products/detail/sparkfun-electronics/DEV-20359/16688101"
+			(at 119.38 62.23 0)
+			(effects
+				(font
+					(size 1.27 1.27)
+				)
+				(hide yes)
+			)
+		)
 		(pin "2"
 		)
@@
 			)
 		)
+		(property "DIGIKEY LINK" "https://www.digikey.com/en/products/detail/yageo/RC0603FR-0710RL/726879"
+			(at 234.95 105.41 0)
+			(effects
+				(font
+					(size 1.27 1.27)
+				)
+				(hide yes)
+			)
+		)
 		(pin "2"
 		)
@@
 			)
 		)
+		(property "DIGIKEY LINK" "https://www.digikey.com/en/products/detail/yageo/RC0603JR-070RL/726675"
+			(at 99.06 116.84 0)
+			(effects
+				(font
+					(size 1.27 1.27)
+				)
+				(hide yes)
+			)
+		)
 		(pin "2"
 		)
@@
 			)
 		)
+		(property "DIGIKEY LINK" "https://www.digikey.com/en/products/detail/yageo/RC0603FR-0710RL/726879"
+			(at 234.95 90.17 0)
+			(effects
+				(font
+					(size 1.27 1.27)
+				)
+				(hide yes)
+			)
+		)
 		(pin "2"
 		)
@@
 			)
 		)
+		(property "DIGIKEY LINK" "https://www.digikey.com/en/products/detail/yageo/RC0603FR-0710RL/726879"
+			(at 234.95 97.79 0)
+			(effects
+				(font
+					(size 1.27 1.27)
+				)
+				(hide yes)
+			)
+		)
 		(pin "2"
 		)
@@
 			)
 		)
+		(property "DIGIKEY LINK" "https://www.digikey.com/en/products/detail/yageo/RC0603FR-0710KL/726880"
+			(at 232.41 57.15 0)
+			(effects
+				(font
+					(size 1.27 1.27)
+				)
+				(hide yes)
+			)
+		)
 		(pin "2"
 		)
@@
 			)
 		)
+		(property "DIGIKEY LINK" "https://www.digikey.com/en/products/detail/keystone-electronics/3034/4499289"
+			(at 45.72 175.26 0)
+			(effects
+				(font
+					(size 1.27 1.27)
+				)
+				(hide yes)
+			)
+		)
 		(pin "1"
 		)
@@
 			)
 		)
+		(property "DIGIKEY LINK" "https://www.digikey.com/en/products/detail/w%C3%BCrth-elektronik/150060GS75000/4489898"
+			(at 259.08 111.76 90)
+			(effects
+				(font
+					(size 1.27 1.27)
+				)
+				(hide yes)
+			)
+		)
 		(pin "2"
 		)
@@
 			)
 		)
+		(property "DIGIKEY LINK" "https://www.digikey.com/en/products/detail/w%C3%BCrth-elektronik/150060BS75000/4489895"
+			(at 250.19 111.76 90)
+			(effects
+				(font
+					(size 1.27 1.27)
+				)
+				(hide yes)
+			)
+		)
 		(pin "2"
 		)
@@
 			(effects
 				(font
+					(size 1.27 1.27)
+				)
+				(hide yes)
+			)
+		)
+		(property "DIGIKEY LINK" "https://www.digikey.com/en/products/detail/w%C3%BCrth-elektronik/150060AS75000/10468254"
+			(at 241.3 111.76 90)
+			(effects
+				(font
