File: gyro.kicad_sch (KiCad schematic)
At the start: 14 parts, among them U102 BNO055, Y100 ABS07-32.768KHZ-T

Commit message: finished up schematic, added magnetic sensor, cleaned up pins, etc.
Parts:
- C116, C117: footprint Capacitor_SMD:C_0805_2012Metric_Pad1.18x1.45mm_HandSolder -> Capacitor_SMD:C_0603_1608Metric_Pad1.08x0.95mm_HandSolder; Digikey https://www.digikey.com/en/products/detail/murata-electroni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 -> (none)
- C118, C119: Digikey https://www.digikey.com/en/products/detail/murata-electroni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 -> (none)
Changed lines of the file:
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@@
-			)
-		)
-		(property "Digikey" "https://www.digikey.com/en/products/detail/murata-electronics/GCM21BR72A104KA37L/1641663"
-			(at 156.21 147.32 0)
-			(effects
-				(font
-					(size 1.27 1.27)
-				)
-				(hide yes)
 			)
 		)
@@
 			)
 		)
-		(property "Footprint" "Capacitor_SMD:C_0805_2012Metric_Pad1.18x1.45mm_HandSolder"
+		(property "Footprint" "Capacitor_SMD:C_0603_1608Metric_Pad1.08x0.95mm_HandSolder"
 			(at 176.53 82.2452 0)
 			(effects
@@
 		)
 		(property "Description" "Unpolarized capacitor"
-			(at 180.34 81.28 0)
-			(effects
-				(font
-					(size 1.27 1.27)
-				)
-				(hide yes)
-			)
-		)
-		(property "Digikey" "https://www.digikey.com/en/products/detail/murata-electronics/GCM21BR72A104KA37L/1641663"
 			(at 180.34 81.28 0)
 			(effects
@@
 			)
 		)
-		(property "Footprint" "Capacitor_SMD:C_0805_2012Metric_Pad1.18x1.45mm_HandSolder"
+		(property "Footprint" "Capacitor_SMD:C_0603_1608Metric_Pad1.08x0.95mm_HandSolder"
 			(at 115.57 110.1852 0)
 			(effects
@@
 		)
 		(property "Description" "Unpolarized capacitor"
-			(at 119.38 109.22 0)
-			(effects
-				(font
-					(size 1.27 1.27)
-				)
-				(hide yes)
-			)
-		)
-		(property "Digikey" "https://www.digikey.com/en/products/detail/murata-electronics/GCM21BR72A104KA37L/1641663"
 			(at 119.38 109.22 0)
 			(effects
@@
 			(at 135.89 147.32 0)
 			(effects
-				(font
-					(size 1.27 1.27)
-				)
-				(hide yes)
-			)
-		)
-		(property "Digikey" "https://www.digikey.com/en/products/detail/murata-electronics/GCM21BR72A104KA37L/1641663"
-			(at 135.89 147.32 0)
-			(effects

Commit message: added TVS diodes to external pins for protection. Ran fabrication output. Ran iBOM generation. All part links can be seen in the iBOM. Download and open to see this
Parts:
- C116, C117, C118, C119: DIGIKEY LINK (none) -> https://www.digikey.com/en/products/detail/murata-electroni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
- R130, R131, R132: DIGIKEY LINK (none) -> https://www.digikey.com/en/products/detail/yageo/RC0603JR-0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
- R133, R134, R135: DIGIKEY LINK (none) -> https://www.digikey.com/en/products/detail/yageo/RC0603FR-0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
- U102: DIGIKEY LINK (none) -> https://www.digikey.com/en/products/detail/bosch-sensortec/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
- Y100: DIGIKEY LINK (none) -> https://www.digikey.com/en/products/detail/abracon-llc/ABS0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
Changed lines of the file:
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@@
 	(generator_version "8.0")
 	(paper "A4")
+	(title_block
+		(date "2025-02-11")
+	)
 	(junction
 		(at 173.99 81.28)
@@
 			)
 		)
+		(property "DIGIKEY LINK" "https://www.digikey.com/en/products/detail/murata-electronics/GRM1885C1H220JA01D/586912"
+			(at 156.21 147.32 0)
+			(effects
+				(font
+					(size 1.27 1.27)
+				)
+				(hide yes)
+			)
+		)
 		(pin "2"
 		)
@@
 			)
 		)
+		(property "DIGIKEY LINK" "https://www.digikey.com/en/products/detail/bosch-sensortec/BNO055/6136301"
+			(at 146.05 93.98 0)
+			(effects
+				(font
+					(size 1.27 1.27)
+				)
+				(hide yes)
+			)
+		)
 		(pin "15"
 		)
@@
 			)
 		)
+		(property "DIGIKEY LINK" "https://www.digikey.com/en/products/detail/yageo/RC0603FR-0710KL/726880"
+			(at 119.38 104.14 0)
+			(effects
+				(font
+					(size 1.27 1.27)
+				)
+				(hide yes)
+			)
+		)
 		(pin "2"
 		)
@@
 		)
 		(property "Description" "Resistor"
+			(at 180.34 99.06 0)
+			(effects
+				(font
+					(size 1.27 1.27)
+				)
+				(hide yes)
+			)
+		)
+		(property "DIGIKEY LINK" "https://www.digikey.com/en/products/detail/yageo/RC0603JR-070RL/726675"
 			(at 180.34 99.06 0)
 			(effects
@@
 			)
 		)
+		(property "DIGIKEY LINK" "https://www.digikey.com/en/products/detail/yageo/RC0603JR-070RL/726675"
+			(at 171.45 104.14 0)
+			(effects
+				(font
+					(size 1.27 1.27)
+				)
+				(hide yes)
+			)
+		)
 		(pin "2"
 		)
@@
 			)
 		)
+		(property "DIGIKEY LINK" "https://www.digikey.com/en/products/detail/murata-electronics/GCJ188R71E104KA12D/7363221"
+			(at 180.34 81.28 0)
+			(effects
+				(font
+					(size 1.27 1.27)
+				)
+				(hide yes)
+			)
+		)
 		(pin "2"
 		)
@@
 			)
 		)
+		(property "DIGIKEY LINK" "https://www.digikey.com/en/products/detail/murata-electronics/GCJ188R71E104KA12D/7363221"
+			(at 119.38 109.22 0)
+			(effects
+				(font
+					(size 1.27 1.27)
+				)
+				(hide yes)
+			)
+		)
 		(pin "2"
 		)
@@
 		)
 		(property "Description" "Resistor"
+			(at 119.38 83.82 0)
+			(effects
+				(font
+					(size 1.27 1.27)
+				)
+				(hide yes)
+			)
+		)
+		(property "DIGIKEY LINK" "https://www.digikey.com/en/products/detail/yageo/RC0603FR-0710KL/726880"
 			(at 119.38 83.82 0)
 			(effects
@@
 			)
 		)
+		(property "DIGIKEY LINK" "https://www.digikey.com/en/products/detail/abracon-llc/ABS07-32-768KHZ-T/1236858"
+			(at 146.05 137.16 0)
+			(effects
+				(font
+					(size 1.27 1.27)
+				)
+				(hide yes)
+			)
+		)
 		(pin "1"
 		)
@@
 		)
 		(property "Description" "Unpolarized capacitor"
+			(at 135.89 147.32 0)
+			(effects
+				(font
+					(size 1.27 1.27)
+				)
+				(hide yes)
+			)
+		)
+		(property "DIGIKEY LINK" "https://www.digikey.com/en/products/detail/murata-electronics/GRM1885C1H220JA01D/586912"
 			(at 135.89 147.32 0)
 			(effects
@@
 			)
 		)
+		(property "DIGIKEY LINK" "https://www.digikey.com/en/products/detail/yageo/RC0603JR-070RL/726675"
+			(at 175.26 101.6 0)
+			(effects
+				(font
+					(size 1.27 1.27)
+				)
+				(hide yes)
+			)
+		)
 		(pin "2"
 		)
@@
 			(at 119.38 81.28 0)
 			(effects
+				(font
+					(size 1.27 1.27)
+				)
+				(hide yes)
+			)
+		)
+		(property "DIGIKEY LINK" "https://www.digikey.com/en/products/detail/yageo/RC0603FR-0710KL/726880"
+			(at 119.38 81.28 0)
+			(effects
